File: Hardware/60_percent_keyboard.kicad_pcb (KiCad board)
At the start: 2 copper layers, 233.8 x 81.8 mm, 100 parts, among them J1 Conn_01x02_Socket, SW1 SW_SPDT, SW2 SW_Push, U1 nice_nano

Commit message: testing to see if it still compiles
Other:
- board text added: "hxw: 81.75 X 233.750 mm curve radius: 2.75 mm"
Changed lines of the file:
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@@
     (effects (font (size 1 1) (thickness 0.15)) (justify left bottom))
+  )
+  (gr_text "hxw: 81.75 X 233.750 mm \ncurve radius: 2.75 mm\n\n\n" (at 56.75 175.75) (layer "User.1")
+    (effects (font (size 5 5) (thickness 0.5)) (justify left bottom))
   )
   (segment (start 61.8 69.75) (end 63.855 69.75) (width 0.5) (layer "F.Cu") (net 4))
